File: pcb/activeSuspension/activeSuspension.kicad_sch (KiCad schematic)
At the start: 18 parts, among them J1 TOF Front Left, J10 TOF Back Right, J11 Conn_01x06_Pin, J12 Conn_01x06_Pin, J13 TOF Back Right, J14 TOF Back Right, J15 Conn_01x02_Pin, J16 Conn_01x02_Pin, J17 Conn_01x04_Pin, J2 TOF Front Right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

Commit message: UPDATED
Parts:
- removed J11, J12, J8, J9: Conn_01x06_Pin, symbol Connector:Conn_01x06_Pin
- removed J15: Conn_01x02_Pin, symbol Connector:Conn_01x02_Pin
- added J11: Servo Front Right, Connector_PinHeader_2.54mm:PinHeader_1x03_P2.54mm_Vertical, symbol Connector:Conn_01x03_Pin
- added J12, J25, J30, J31, J33, J8: HX711 Front Left, Connector_PinHeader_2.54mm:PinHeader_1x04_P2.54mm_Vertical, symbol Connector:Conn_01x04_Pin
- added J15: Back motors control, Connector_PinHeader_2.54mm:PinHeader_1x06_P2.54mm_Vertical, symbol Connector:Conn_01x06_Pin
- added J18: Back motors power, TerminalBlock_MetzConnect:TerminalBlock_MetzConnect_Type101_RT01602HBWC_1x02_P5.08mm_Horizontal, symbol Connector:Conn_01x02_Pin
- added J19: Front motors control, Connector_PinHeader_2.54mm:PinHeader_1x06_P2.54mm_Vertical, symbol Connector:Conn_01x06_Pin
- added J20: Front motors power, TerminalBlock_MetzConnect:TerminalBlock_MetzConnect_Type101_RT01602HBWC_1x02_P5.08mm_Horizontal, symbol Connector:Conn_01x02_Pin
- added J21, J22, J23, J24: Conn_01x01_Pin, Connector_PinHeader_2.54mm:PinHeader_1x01_P2.54mm_Vertical, symbol Connector:Conn_01x01_Pin
- added J26: MPU6050, Connector_PinHeader_2.54mm:PinHeader_1x04_P2.54mm_Vertical, symbol Connector:Conn_01x04_Pin
- added J27: Servo Front Left, Connector_PinHeader_2.54mm:PinHeader_1x03_P2.54mm_Vertical, symbol Connector:Conn_01x03_Pin
- added J28: Servo Back Right, Connector_PinHeader_2.54mm:PinHeader_1x03_P2.54mm_Vertical, symbol Connector:Conn_01x03_Pin
- added J29: Servo Back Left, Connector_PinHeader_2.54mm:PinHeader_1x03_P2.54mm_Vertical, symbol Connector:Conn_01x03_Pin
- added J32, J9: HX711 Back Left, Connector_PinHeader_2.54mm:PinHeader_1x04_P2.54mm_Vertical, symbol Connector:Conn_01x04_Pin
- J1, J2, J3, J4: footprint (none) -> Connector_PinHeader_2.54mm:PinHeader_1x04_P2.54mm_Vertical
- J10: value TOF Back Right -> HX711 Front Right; footprint (none) -> Connector_PinHeader_2.54mm:PinHeader_1x04_P2.54mm_Vertical
- J13: value TOF Back Right -> HX711 Back Left; footprint (none) -> Connector_PinHeader_2.54mm:PinHeader_1x04_P2.54mm_Vertical
- J14: value TOF Back Right -> HX711 Back Right; footprint (none) -> Connector_PinHeader_2.54mm:PinHeader_1x04_P2.54mm_Vertical
- J16: value Conn_01x02_Pin -> Power in 12V; footprint (none) -> Connector_PinHeader_2.54mm:PinHeader_1x02_P2.54mm_Vertical
- J17: value Conn_01x04_Pin -> FPGA Input; footprint (none) -> Connector_PinHeader_2.54mm:PinHeader_1x04_P2.54mm_Vertical
- J5, J6: footprint (none) -> Connector_PinHeader_2.54mm:PinHeader_1x12_P2.54mm_Vertical
- J7: value TOF Back Right -> HX711 Front Left; footprint (none) -> Connector_PinHeader_2.54mm:PinHeader_1x04_P2.54mm_Vertical
Connections:
- net 12V: now also J18.1 (Pin_1), J20.1 (Pin_1), J21.1 (Pin_1)
- net 3V3: now also J26.1 (Pin_1)
- net DT0: now also U1.J1_5 (GPIO5)
- net DT1: now also U1.J3_10 (GPIO38)
- net DT2: now also U1.J1_6 (GPIO6)
- net DT3: now also U1.J3_15 (GPIO45)
- net FPGA0: now also J17.1 (Pin_1), U1.J3_7 (MTDI/GPIO41)
- net FPGA1: now also J17.2 (Pin_2), U1.J3_8 (MTDO/GPIO40)
- net GND: now also J17.3 (Pin_3), J11.1 (Pin_1), J18.2 (Pin_2), J20.2 (Pin_2), J22.1 (Pin_1), J24.1 (Pin_1), J26.2 (Pin_2), J27.1 (Pin_1), J28.1 (Pin_1), J29.1 (Pin_1)
- net SCK0: now also U1.J1_4 (GPIO4)
- net SCK1: now also U1.J3_9 (MTCK/GPIO39)
- net SCK2: now also U1.J1_7 (GPIO7)
- net SCK3: now also U1.J3_16 (GPIO48)
- net SCL1: now also J4.4 (Pin_4), J6.12 (Pin_12); no longer J2.4 (Pin_4), J5.12 (Pin_12)
- net SCL2: now also J5.12 (Pin_12); no longer J6.12 (Pin_12)
- net SCL3: now also J2.4 (Pin_4); no longer J4.4 (Pin_4)
- net SCL_MPU: now also J26.3 (Pin_3)
- net SDA1: now also J4.3 (Pin_3), J6.11 (Pin_11); no longer J2.3 (Pin_3), J5.11 (Pin_11)
- net SDA2: now also J5.11 (Pin_11); no longer J6.11 (Pin_11)
- net SDA3: now also J2.3 (Pin_3); no longer J4.3 (Pin_3)
- net SDA_MPU: now also J26.4 (Pin_4)
- net EN: now reaches U1.J1_17 (GPIO11)
- net EN: now also J15.1 (Pin_1), J15.6 (Pin_6), J19.1 (Pin_1), J19.6 (Pin_6)
- net PWM0: now reaches U1.J1_18 (GPIO12)
- net PWM0: now also J27.3 (Pin_3)
- net IN1: now reaches U1.J1_19 (GPIO13)
- net IN1: now also J15.2 (Pin_2), J15.4 (Pin_4), J19.3 (Pin_3), J19.5 (Pin_5)
- net IN2: now reaches U1.J1_20 (GPIO14)
- net IN2: now also J15.3 (Pin_3), J15.5 (Pin_5), J19.2 (Pin_2), J19.4 (Pin_4)
- net 5V: now reaches U1.J1_21 (5V0)
- net 5V: now also J17.4 (Pin_4), J11.2 (Pin_2), J23.1 (Pin_1), J27.2 (Pin_2), J28.2 (Pin_2), J29.2 (Pin_2)
- net PWM3: now reaches U1.J3_17 (GPIO47)
- net PWM3: now also J29.3 (Pin_3)
- net PWM2: now reaches U1.J3_18 (GPIO21)
- net PWM2: now also J28.3 (Pin_3)
- net PWM1: now reaches U1.J3_6 (MTMS/GPIO42)
- net PWM1: now also J11.3 (Pin_3)
- new net 0A+: J25.1 (Pin_1), J30.1 (Pin_1)
- new net 0A-: J25.2 (Pin_2), J30.2 (Pin_2)
- new net 0E+: J25.4 (Pin_4), J30.4 (Pin_4)
- new net 0E-: J25.3 (Pin_3), J30.3 (Pin_3)
- new net 1A+: J31.1 (Pin_1), J8.1 (Pin_1)
- new net 1A-: J31.2 (Pin_2), J8.2 (Pin_2)
- new net 1E+: J31.4 (Pin_4), J8.4 (Pin_4)
- new net 1E-: J31.3 (Pin_3), J8.3 (Pin_3)
- new net 2A+: J32.1 (Pin_1), J9.1 (Pin_1)
- new net 2A-: J32.2 (Pin_2), J9.2 (Pin_2)
- new net 2E+: J32.4 (Pin_4), J9.4 (Pin_4)
- new net 2E-: J32.3 (Pin_3), J9.3 (Pin_3)
- new net 3A+: J12.1 (Pin_1), J33.1 (Pin_1)
- new net 3A-: J12.2 (Pin_2), J33.2 (Pin_2)
- new net 3E+: J12.4 (Pin_4), J33.4 (Pin_4)
- new net 3E-: J12.3 (Pin_3), J33.3 (Pin_3)
Other:
- moved on the sheet: J17
