File: pcb/activeSuspension/activeSuspension.kicad_pcb (KiCad board)
At the start: 2 copper layers, 220 x 87.5 mm, 34 parts, among them J1 TOF Front Left, J10 HX711 Front Right, J11 Servo Front Right, J12 HX711 Front Left, J13 HX711 Back Left, J14 HX711 Back Right, J15 Back motors control, J16 Power in 12V, J17 FPGA Input, J18 Back motors power, J19 Front motors control, J2 TOF Front Right, J20 Front motors power, J21 Conn_01x01_Pin, J22 Conn_01x01_Pin, J23 Conn_01x01_Pin, J24 Conn_01x01_Pin, J25 HX711 Front Left, J26 MPU6050, J27 Servo Front Left, J28 Servo Back Right, J29 Servo Back Left, J3 TOF Back Left, J30 HX711 Front Left, J31 HX711 Front Left, J32 HX711 Back Left, J33 HX711 Front Left, J4 TOF Back Right, J5 Conn_01x12_Pin, J6 Conn_01x12_Pin, J7 HX711 Front Left, J8 HX711 Front Left, J9 HX711 Back Left, U1 ESP32-S3-DEVKITC-1-N8R2

Commit message: UPDATED
Routing:
- net PWM0: track 4.10 -> 148.0 mm, vias 0 -> 4
- net EN: track 193.8 -> 201.4 mm
- net GND: track 881.4 -> 874.8 mm
- net SDA_MPU: track 29.8 -> 26.9 mm
- net 5V: track 348.6 -> 351.4 mm
- net SCL_MPU: track 33.9 -> 31.1 mm
- net SDA2: track 189.4 -> 188.4 mm
- net SCL1: track 154.5 -> 154.0 mm
Other:
- board size 220 x 87.5 mm -> 230 x 87.5 mm
- board text added: "0"
- board text added: "1"
- board text added: "3V3"
- board text added: "ACTIVE SUSPENSION SYSTEM"
- board text added: "Multiplexer"

Commit message: updated
Connections:
- U1 pad J3_12: unconnected-(U1-GPIO36-PadJ3_12) -> SCK3
- U1 pad J3_13: unconnected-(U1-GPIO35-PadJ3_13) -> DT3
Routing:
- net SCK3: track 20.1 -> 41.3 mm
- net DT3: track 24.3 -> 32.1 mm
